File: motherboard/fs.kicad_sch (KiCad schematic)
At the start: 87 parts, among them J101 Header, J102 640389-2, Q101 MJD44H11, Q102 MJD45H11, U101 INA132UA, U102 LM741C, U103 LMH6609, U104 LM317, U105 LM337, U106 LM340-5, U107 MC7905ACD2T

Commit message: replace mosfet with analog switch
Parts:
- added C116: 10μF, Capacitor_SMD:C_0805_2012Metric, symbol #SRS:5_Capacitors/5-00954
- added C117, C118, C119, C120: 0.1μF, Capacitor_SMD:C_0603_1608Metric, symbol #SRS:5_Capacitors/5-00764
- added D102: MMBD352, Package_TO_SOT_SMD:SOT-23, symbol #SRS:3_ICs/3-00538
- added J103: Conn_01x05, Connector_PinHeader_2.54mm:PinHeader_1x05_P2.54mm_Vertical, symbol Connector_Generic:Conn_01x05
- added Q103: 2N7002, Package_TO_SOT_SMD:SOT-23, symbol Transistor_FET:2N7002
- added R116: 10.0K, Resistor_SMD:R_0603_1608Metric, symbol #SRS:4_Resistors/4-02253
- added R117, R120: 1.00K, Resistor_SMD:R_0603_1608Metric, symbol #SRS:4_Resistors/4-02157
- added R118, R119: 4.99K, Resistor_SMD:R_0603_1608Metric, symbol #SRS:4_Resistors/4-02224
- added U108: DG419DY, Package_SO:SO-8_3.9x4.9mm_P1.27mm, symbol #SRS:3_ICs/3-01367
- D101: value MBRS230LT3G -> MMBD352LT1G
Connections:
- net +5V: now also C117.2, C118.2, C120.2, D102.2 (K), J103.1 (Pin_1), U108.4 (V+), U108.5 (VL)
- net -12V: now also C119.2, U108.7 (V-)
- net GND: now also C116.2, C117.1, C118.1, C119.1, C120.1, D102.1 (A), Q103.2 (S), R120.1, U108.3 (GND)
- net Phase Noise/FREQ_CTL: now also D102.3 (COM)
- net at U101.5 (SENSE), U101.6: now also U108.1; no longer R102.2
- net FREQ_CTL renamed SC10L_FREQ_CTL
- new net: R102.2, U108.2
- new net: C116.1, Q103.1 (G), R116.2
- new net: J103.5 (Pin_5), R120.2
- new net: J103.2 (Pin_2), R117.2
- new net: J103.3 (Pin_3), R118.2
- new net: J103.4 (Pin_4), R119.2
- new net: Q103.3 (D), R117.1
- new net LOCKED: R116.1
- new net ~{OVLD}: R118.1
- new net ~{SIG_PRESENT}: R119.1, U108.6
- no-connect marks 2 -> 3
Other:
- sheet Phase Noise ports: added LOCKED, ~{OVLD}, ~{SIG_PRESENT}; removed none
- note added: "CLAMP TO RANGE (−0.25, +5.25) V"
- note added: "DISCONNECT EFC WHEN EXT 10 MHz NOT PRESENT"
- note added: "MATES TO LED BOARD 7-01993 WITH GREEN/GREEN/GREEN/RED LEDS INSTALLED, VIA SHORT 5 POS RIBBON CABLE (1-01043)"
- moved on the sheet: C101, C102, C103, C104, C105, C106, C107, C108, C109, C110, C111, C112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

Commit message: better comparators for ~FAULT
Parts:
- removed C116: 10μF, Capacitor_SMD:C_0805_2012Metric, symbol #SRS:5_Capacitors/5-00954
- removed J103: Conn_01x05, Connector_PinHeader_2.54mm:PinHeader_1x05_P2.54mm_Vertical, symbol Connector_Generic:Conn_01x05
- removed Q103: 2N7002, Package_TO_SOT_SMD:SOT-23, symbol Transistor_FET:2N7002
- removed R102, R117, R120: 1.00K, Resistor_SMD:R_0603_1608Metric, symbol #SRS:4_Resistors/4-02157
- removed R116: 10.0K, Resistor_SMD:R_0603_1608Metric, symbol #SRS:4_Resistors/4-02253
- removed R118, R119: 4.99K, Resistor_SMD:R_0603_1608Metric, symbol #SRS:4_Resistors/4-02224
- removed U102: LM741C, Package_SO:SO-8_3.9x4.9mm_P1.27mm, symbol #SRS:3_ICs/3-00729
- added R102: 100R, Resistor_SMD:R_0603_1608Metric, symbol #SRS:4_Resistors/4-02061
- added R116: 1.00K, Resistor_SMD:R_0603_1608Metric, symbol #SRS:4_Resistors/4-02157
- added RV101: 10k, Connector_PinHeader_2.54mm:PinHeader_1x03_P2.54mm_Vertical, symbol Device:R_Potentiometer_US
- added U109, U110: NCS20071, Package_TO_SOT_SMD:TSOT-23-5, symbol #SRS:3_ICs/3-02713
- D101: value MMBD352LT1G -> MBRS230LT3G; MPN MBRS230LT3G -> MBRS230LT3G
- D102: value MMBD352 -> MMBD352LT1G
Connections:
- net +12V: now also U110.5 (V+)
- net -12V: now also RV101.3, U109.2 (V-), U110.2 (V-)
- net GND: now also U109.5 (V+)
- net SC10L_+5VREF: now also RV101.1
- net SC10L_FREQ_CTL: now also R102.1
- net at U101.5 (SENSE), U101.6: now also U108.2; no longer U108.1
- net at U108.8: now also R116.2
- net at C103.2, Q101.1 (B), Q102.1 (B)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: now also U110.1
- net at C103.1, R103.2: now also U110.4 (-)
- net at R105.2, R106.1: now also U110.3 (+)
- new net: R102.2, U108.1
- new net: RV101.2, U109.3 (+)
- new net: R116.1, U109.1, U109.4 (-)
- no-connect marks 3 -> 0
Other:
- added sheet Front Panel (fp.kicad_sch)
- sheet Phase Noise ports: added ~{FAULT}, ~{LOCKED}; removed LOCKED, ~{OVLD}
- note added: "(POT ON SEPARATE PCB)"
- note added: "WHEN EXT 10 MHz NOT PRESENT, DISCONNECT EFC AND USE MANUAL ADJUST"
- note removed: "DISCONNECT EFC WHEN EXT 10 MHz NOT PRESENT"
- note removed: "MATES TO LED BOARD 7-01993 WITH GREEN/GREEN/GREEN/RED LEDS INSTALLED, VIA SHORT 5 POS RIBBON CABLE (1-01043)"
- moved on the sheet: C101, C102, C103, C104, C105, C106, C107, C108, C109, C110, C111, C112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

Commit message: female header moved 5 mil away from male header
Parts:
- C106: JLCPCB EEU-FC1V331 -> C14745
