File: ocxo_mount/ocxo_mount.kicad_sch (KiCad schematic)
At the start: 10 parts, among them J1 12POS 2.54MM, J2 Conn_01x12, M1 MountingPad_4-40, M2 MountingPad_4-40, M3 MountingPad_4-40, M4 MountingPad_4-40, M5 MountingPad_4-40, M6 MountingPad_4-40, M7 MountingPad_4-40, M8 MountingPad_4-40

Commit message: add mechanical parts to bom
Parts:
- added PCB101: PCB, symbol GRAPHICAL_SRS:PCB
- added SC1, SC2, SC3, SC4, SC5, SC6, SC7, SC8: 4-40X1/4PP, symbol HARDWARE_SRS:SCREW
- added ST1, ST2, ST3, ST4: 4-40X5/8 HX F/F, symbol HARDWARE_SRS:STANDOFF_F-F
Other:
- note added: "HEX STANDOFFS"
- note added: "SIGNAL_GROUND"

Commit message: fix annotations
Parts:
- J1: value 12POS 2.54MM -> 12POS 2.54mm; Footprint Modified By assignment_engine -> (none); Footprint Modified Timestamp 2025-10-13 21:00:08 -0800 -> (none); Manf Samtec -> (none); Price 0.71 -> (none); Qty In Stock 531 -> (none); Recommended Y -> (none); Symbol Connector_Generic:Conn_01x12 -> (none); Symbol Modified By assignment_engine -> (none); Symbol Modified Timestamp 2025-10-13 21:00:08 -0800 -> (none); Used In CG635,DG645,FS740,SC10L,SG382,SG382R,SG384,SG384R,SG386,SG3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 -> (none)
- J2: MPN (none) -> 1-215299-2; SRS P/N 1-01602 -> (none); SRS PN (none) -> 1-01602
Changed lines of the file:
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@@
 			)
 		)
-		(property "SRS P/N" "1-01602"
-			(at 220.218 95.504 0)
+		(property "MPN" "1-215299-2"
+			(at 213.36 90.17 0)
+			(hide yes)
+			(show_name no)
+			(do_not_autoplace no)
+			(effects
+				(font
+					(size 1.27 1.27)
+				)
+			)
+		)
+		(property "SRS PN" "1-01602"
+			(at 213.36 90.17 0)
+			(hide yes)
 			(show_name no)
 			(do_not_autoplace no)
@@
 			)
 		)
-		(property "Value" "12POS 2.54MM"
+		(property "Value" "12POS 2.54mm"
 			(at 162.56 92.7099 0)
 			(show_name no)
@@
 		)
 		(property "Description" "Conn Unshrouded Header HDR 12 POS 2.54mm Solder ST Thru-Hole Bulk"
-			(at 165.1 90.17 0)
-			(hide yes)
-			(show_name no)
-			(do_not_autoplace no)
-			(effects
-				(font
-					(size 1.27 1.27)
-				)
-			)
-		)
-		(property "Current" ""
-			(at 165.1 90.17 0)
-			(hide yes)
-			(show_name no)
-			(do_not_autoplace no)
-			(effects
-				(font
-					(size 1.27 1.27)
-				)
-			)
-		)
-		(property "Shiny Info" ""
-			(at 165.1 90.17 0)
-			(hide yes)
-			(show_name no)
-			(do_not_autoplace no)
-			(effects
-				(font
-					(size 1.27 1.27)
-				)
-			)
-		)
-		(property "Tempco" ""
-			(at 165.1 90.17 0)
-			(hide yes)
-			(show_name no)
-			(do_not_autoplace no)
-			(effects
-				(font
-					(size 1.27 1.27)
-				)
-			)
-		)
-		(property "Tolerance" ""
-			(at 165.1 90.17 0)
-			(hide yes)
-			(show_name no)
-			(do_not_autoplace no)
-			(effects
-				(font
-					(size 1.27 1.27)
-				)
-			)
-		)
-		(property "Price" "0.71"
 			(at 165.1 90.17 0)
 			(hide yes)
@@
 			)
 		)
-		(property "Footprint Modified Timestamp" "2025-10-13 21:00:08 -0800"
-			(at 165.1 90.17 0)
-			(hide yes)
-			(show_name no)
-			(do_not_autoplace no)
-			(effects
-				(font
-					(size 1.27 1.27)
-				)
-			)
-		)
-		(property "Symbol Modified Timestamp" "2025-10-13 21:00:08 -0800"
-			(at 165.1 90.17 0)
-			(hide yes)
-			(show_name no)
-			(do_not_autoplace no)
-			(effects
-				(font
-					(size 1.27 1.27)
-				)
-			)
-		)
-		(property "Qty In Stock" "531"
-			(at 165.1 90.17 0)
-			(hide yes)
-			(show_name no)
-			(do_not_autoplace no)
-			(effects
-				(font
-					(size 1.27 1.27)
-				)
-			)
-		)
-		(property "Used In" "CG635,DG645,FS740,SC10L,SG382,SG382R,SG384,SG384R,SG386,SG386R,SG392,SG394,SG396"
-			(at 165.1 90.17 0)
-			(hide yes)
-			(show_name no)
-			(do_not_autoplace no)
-			(effects
-				(font
-					(size 1.27 1.27)
-				)
-			)
-		)
-		(property "Symbol" "Connector_Generic:Conn_01x12"
-			(at 165.1 90.17 0)
-			(hide yes)
-			(show_name no)
-			(do_not_autoplace no)
-			(effects
-				(font
-					(size 1.27 1.27)
-				)
-			)
-		)
 		(property "MPN" "HMTSW-112-22-L-S-440-LL"
 			(at 165.1 90.17 0)
@@
 			(at 165.1 90.17 0)
 			(hide yes)
-			(show_name no)
-			(do_not_autoplace no)
-			(effects
-				(font
-					(size 1.27 1.27)
-				)
-			)
-		)
-		(property "Manf" "Samtec"
-			(at 165.1 90.17 0)
-			(hide yes)
-			(show_name no)
-			(do_not_autoplace no)
-			(effects
-				(font
-					(size 1.27 1.27)
-				)
-			)
-		)
-		(property "Recommended" "Y"
-			(at 165.1 90.17 0)
-			(hide yes)
-			(show_name no)
-			(do_not_autoplace no)
-			(effects
-				(font
-					(size 1.27 1.27)
-				)
-			)
-		)
-		(property "Footprint Modified By" "assignment_engine"
-			(at 165.1 90.17 0)
-			(hide yes)
-			(show_name no)
-			(do_not_autoplace no)
-			(effects
-				(font
-					(size 1.27 1.27)
-				)
-			)
-		)
-		(property "Symbol Modified By" "assignment_engine"
-			(at 165.1 90.17 0)
-			(hide yes)

Commit message: female header moved 5 mil away from male header
Changed lines of the file:
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@@
 		)
 		(property "SRS PN" "1-01602"
-			(at 213.36 90.17 0)
-			(hide yes)
+			(at 220.726 95.25 0)
 			(show_name no)
 			(do_not_autoplace no)
